File: PCB/Galia.kicad_sch (KiCad schematic)
At the start: 10 parts, among them J1 USB In, J2 Power, J3 I/O, SW1 PTS45, SW2 PTS45, U1 TPD4E05U06

Commit message: 26/07/2023 update
Fixed position of button and mounting holes. Added JLC tooling holes.
Parts:
- added H3, H4, H5: Tooling Hole, Galia:JLC Tooling Hole, symbol Mechanical:MountingHole
- SW1, SW2: value PTS45 -> PTS645
Changed lines of the file:
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@@
+    )
+  )
+  (symbol (lib_id "Mechanical:MountingHole") (at 175.26 55.88 0) (unit 1)
+    (in_bom no) (on_board yes) (dnp no)
+    (property "Reference" "H5" (at 177.8 54.7116 0)
+      (effects (font (size 1.27 1.27)) (justify left))
+    )
+    (property "Value" "Tooling Hole" (at 177.8 57.023 0)
+      (effects (font (size 1.27 1.27)) (justify left))
+    )
+    (property "Footprint" "Galia:JLC Tooling Hole" (at 175.26 55.88 0)
+      (effects (font (size 1.27 1.27)) hide)
+    )
+    (property "Datasheet" "" (at 175.26 55.88 0)
+      (effects (font (size 1.27 1.27)) hide)
+    )
+    (property "LCSC" "" (at 175.26 55.88 0)
+      (effects (font (size 1.27 1.27)) hide)
+    )
+    (instances
+      (project "Galia"
+        (path "/1215eee5-143d-4cdd-be21-2ea99cea4a06"
+          (reference "H5") (unit 1)
+        )
+      )
+      (project "Honeydew"
+        (path "/534caec7-cf60-4f90-b1ed-42c9d445ef0f"
+          (reference "H3") (unit 1)
+        )
+      )
+      (project "Crenshaw"
+        (path "/e15cb478-ed36-448a-aade-2c525821f2a0"
+          (reference "H4") (unit 1)
+        )
+      )
     )
   )
@@
       (effects (font (size 1.27 1.27)))
     )
-    (property "Value" "PTS45" (at 129.54 20.32 0)
+    (property "Value" "PTS645" (at 129.54 20.32 0)
       (effects (font (size 1.27 1.27)))
     )
@@
         (path "/534caec7-cf60-4f90-b1ed-42c9d445ef0f/d133c1c6-f35d-4b98-81a0-3607ab1d2de1"
           (reference "SW68") (unit 1)
+        )
+      )
+    )
+  )
+  (symbol (lib_id "Mechanical:MountingHole") (at 175.26 45.72 0) (unit 1)
+    (in_bom no) (on_board yes) (dnp no)
+    (property "Reference" "H3" (at 177.8 44.5516 0)
+      (effects (font (size 1.27 1.27)) (justify left))
+    )
+    (property "Value" "Tooling Hole" (at 177.8 46.863 0)
+      (effects (font (size 1.27 1.27)) (justify left))
+    )
+    (property "Footprint" "Galia:JLC Tooling Hole" (at 175.26 45.72 0)
+      (effects (font (size 1.27 1.27)) hide)
+    )
+    (property "Datasheet" "" (at 175.26 45.72 0)
+      (effects (font (size 1.27 1.27)) hide)
+    )
+    (property "LCSC" "" (at 175.26 45.72 0)
+      (effects (font (size 1.27 1.27)) hide)
+    )
+    (instances
+      (project "Galia"
+        (path "/1215eee5-143d-4cdd-be21-2ea99cea4a06"
+          (reference "H3") (unit 1)
+        )
+      )
+      (project "Honeydew"
+        (path "/534caec7-cf60-4f90-b1ed-42c9d445ef0f"
+          (reference "H1") (unit 1)
+        )
+      )
+      (project "Crenshaw"
+        (path "/e15cb478-ed36-448a-aade-2c525821f2a0"
+          (reference "H2") (unit 1)
         )
       )
@@
         (path "/534caec7-cf60-4f90-b1ed-42c9d445ef0f/03fe79d8-f43d-4879-be7c-5a505456d728"
           (reference "#PWR041") (unit 1)
+        )
+      )
+    )
+  )
+  (symbol (lib_id "Mechanical:MountingHole") (at 175.26 50.8 0) (unit 1)
+    (in_bom no) (on_board yes) (dnp no)
+    (property "Reference" "H4" (at 177.8 49.6316 0)
+      (effects (font (size 1.27 1.27)) (justify left))
+    )
+    (property "Value" "Tooling Hole" (at 177.8 51.943 0)
+      (effects (font (size 1.27 1.27)) (justify left))
+    )
+    (property "Footprint" "Galia:JLC Tooling Hole" (at 175.26 50.8 0)
+      (effects (font (size 1.27 1.27)) hide)
+    )
+    (property "Datasheet" "" (at 175.26 50.8 0)
+      (effects (font (size 1.27 1.27)) hide)
+    )
+    (property "LCSC" "" (at 175.26 50.8 0)
+      (effects (font (size 1.27 1.27)) hide)
+    )
+    (instances
+      (project "Galia"
+        (path "/1215eee5-143d-4cdd-be21-2ea99cea4a06"
+          (reference "H4") (unit 1)
+        )
+      )
+      (project "Honeydew"
+        (path "/534caec7-cf60-4f90-b1ed-42c9d445ef0f"
+          (reference "H2") (unit 1)
+        )
+      )
+      (project "Crenshaw"
+        (path "/e15cb478-ed36-448a-aade-2c525821f2a0"
+          (reference "H3") (unit 1)
         )
       )
@@
       (effects (font (size 1.27 1.27)))
     )
-    (property "Value" "PTS45" (at 129.54 33.02 0)
-      (effects (font (size 1.27 1.27)))
-    )
+    (property "Value" "PTS645" (at 129.54 33.02 0)
+      (effects (font (size 1.27 1.27)))
+    )
